Commit message: Created some class files to the wall follwer algorith

File: files/catkin_ws/src/one_kinect_robot/urdf/kinect_robot.xacro (robot description, xacro)
@@ -10,5 +10,5 @@
       <mass value="5"/>
       <origin rpy="0 0 0" xyz="0 0 0.1"/>
-      <inertia ixx="0.0395416666667" ixy="0" ixz="0" iyy="0.106208333333" iyz="0" izz="0.106208333333"/>
+      <inertia ixx="0.0395416666667" ixy="0" ixz="0" iyy="0.106208333333" iyz="0" izz="0.141666667"/>
     </inertial>
     <!-- body -->
@@ -52,6 +52,6 @@
     <inertial>
         <origin xyz="0 0 0" rpy="0 0 0" />
-        <mass value="1" />
-        <xacro:cube_inertia mass="1" w="0.05" h="0.05" d="0.05" />
+        <mass value="3" />
+        <xacro:cube_inertia mass="3" w="0.05" h="0.05" d="0.05" />
     </inertial>
     <visual>
